Commit message: modify robot xacro for conversion to sdf

File: config/urdf/r2b2.xacro (robot description, xacro)
@@ -1,4 +1,4 @@
 <?xml version="1.0"?>
-<robot name="B2" xmlns:xacro="http://ros.org/wiki/xacro">
+<robot name="R2B2" xmlns:xacro="http://ros.org/wiki/xacro">
     <!-- Configurable Measurements -->
     <xacro:property name="wheel_dia" value="0.064" />
@@ -10,10 +10,37 @@
     <xacro:property name="base_plate_ht" value="0.006" />
     <xacro:property name="base_standoff_ht" value="0.060" />
+    <xacro:property name="base_link_mass" value="2.285" />
     <xacro:property name="motor_mount_ht" value="0.0145" />
     <xacro:property name="sensor_arch_ht" value="0.062" />
+    <xacro:property name="camera_length" value="0.025" />
+    <xacro:property name="camera_width" value="0.090" />
+    <xacro:property name="camera_height" value="0.025" />
+    <xacro:property name="camera_mass" value="0.069" />
+    <xacro:property name="scanner_box_length" value="0.0968" />
+    <xacro:property name="scanner_box_width" value="0.0703" />
+    <xacro:property name="scanner_box_height" value="0.055" />
+    <xacro:property name="scanner_mass" value="0.170" />
+    <xacro:property name="imu_length" value="0.02032" />
+    <xacro:property name="imu_width" value="0.0127" />
+    <xacro:property name="imu_height" value="0.003" />
+    <xacro:property name="imu_mass" value="0.0007" />
     <!-- Derived Measurements -->
     <xacro:property name="base_box_ht" value="${base_plate_ht + base_standoff_ht + base_plate_ht}" />
     <xacro:property name="base_box_ht_from_floor" value="${wheel_dia/2 + motor_mount_ht}"/>
     <xacro:property name="base_box_top_ht" value="${base_box_ht_from_floor + base_box_ht}"/>
+    <!-- Macros -->
+    <xacro:macro name="box_inertial" params="mass length width height">
+        <inertial>
+            <mass value="${mass}" />
+            <inertia
+                ixx="${1/12 * mass * (pow(height, 2) + pow(length, 2))}"
+                ixy="0"
+                ixz="0"
+                iyy="${1/12 * mass * (pow(width, 2) + pow(height, 2))}"
+                iyz="0"
+                izz="${1/12 * mass * (pow(width, 2) + pow(length, 2))}"
+            />
+        </inertial>
+    </xacro:macro>
     <!-- Joints -->
     <joint name="camera_link_joint" type="fixed">
@@ -22,5 +49,5 @@
         <child link="camera_link"/>
     </joint>
-    <joint name="imu_link_join" type="fixed">
+    <joint name="imu_link_joint" type="fixed">
         <origin xyz="0.040 -0.040 ${base_box_top_ht + sensor_arch_ht + 0.008}"
                 rpy="0.0 0.0 0.0"/>
@@ -42,4 +69,7 @@
             <origin xyz="0.0 0.0 ${base_box_ht_from_floor + base_box_ht/2}"/>
             <material name="White" />
+            <gazebo reference="frame_box">
+                <material>Gazebo/White</material>
+            </gazebo>
         </visual>
         <visual name="nuc">
@@ -51,4 +81,7 @@
             <origin xyz="-0.0335 0.0 ${base_box_top_ht + 0.036/2}"/>
             <material name="White" />
+            <gazebo reference="nuc">
+                <material>Gazebo/White</material>
+            </gazebo>
         </visual>
         <visual name="raspberry_pi4">
@@ -58,4 +91,7 @@
             <origin xyz="0.077 0.0 ${base_box_top_ht + 0.030/2}"/>
             <material name="White" />
+            <gazebo reference="raspberry_pi4">
+                <material>Gazebo/White</material>
+            </gazebo>
         </visual>
         <!-- Wheels -->
@@ -66,4 +102,7 @@
             <origin xyz="${wheel_x_from_ctr} ${wheel_y_from_ctr} ${wheel_dia/2}" rpy="${pi/2} 0.0 0.0"/>
             <material name="Black" />
+            <gazebo reference="front_left_wheel">
+                <material>Gazebo/Black</material>
+            </gazebo>
         </visual>
         <visual name="front_right_wheel">
@@ -73,4 +112,7 @@
             <origin xyz="${wheel_x_from_ctr} -${wheel_y_from_ctr} ${wheel_dia/2}" rpy="${pi/2} 0.0 0.0"/>
             <material name="Black" />
+            <gazebo reference="front_right_wheel">
+                <material>Gazebo/Black</material>
+            </gazebo>
         </visual>
         <visual name="rear_left_wheel">
@@ -80,4 +122,7 @@
             <origin xyz="-${wheel_x_from_ctr} ${wheel_y_from_ctr} ${wheel_dia/2}" rpy="${pi/2} 0.0 0.0"/>
             <material name="Black" />
+            <gazebo reference="rear_left_wheel">
+                <material>Gazebo/Black</material>
+            </gazebo>
         </visual>
         <visual name="rear_right_wheel">
@@ -87,21 +132,44 @@
             <origin xyz="-${wheel_x_from_ctr} -${wheel_y_from_ctr} ${wheel_dia/2}" rpy="${pi/2} 0.0 0.0"/>
             <material name="Black" />
-        </visual>
+            <gazebo reference="rear_right_wheel">
+                <material>Gazebo/Black</material>
+            </gazebo>
+        </visual>
+        <collision>
+            <geometry>
+                <box size="${base_x_len} ${base_y_width} ${base_box_ht}"/>
+            </geometry>
+        </collision>
+        <xacro:box_inertial
+            mass="${base_link_mass}" length="${base_x_len}"
+            width="${base_y_width}" height="${base_box_ht}" />
     </link>
     <link name="camera_link">
         <visual>
         <geometry>
-            <box size="0.025 0.085 0.025"/>
+            <box size="${camera_length}, ${camera_width} ${camera_height}"/>
         </geometry>
         <material name="Sky Blue" />
-        </visual>
+        <gazebo reference="camera_link">
+            <material>Gazebo/Blue</material>
+        </gazebo>
+    </visual>
+        <xacro:box_inertial
+            mass="${camera_mass}" length="${camera_length}"
+            width="${camera_width}" height="${camera_height}" />
     </link>
     <link name="imu_link">
         <visual>
             <geometry>
-                <box size="0.02032 0.0127 0.003"/>
+                <box size="${imu_length} ${imu_width} ${imu_height}" />
             </geometry>
             <material name="PCB Green" />
-        </visual>
+            <gazebo reference="imu_link">
+                <material>Gazebo/Green</material>
+            </gazebo>
+        </visual>
+        <xacro:box_inertial
+            mass="${imu_mass}" length="${imu_length}"
+            width="${imu_width}" height="${imu_height}" />
     </link>
     <link name="scanner_link">
@@ -125,5 +193,11 @@
             <origin xyz="0.015 0.0 -0.033"/>
             <material name="Black" />
-        </visual>
+            <gazebo reference="scanner_link">
+                <material>Gazebo/Black</material>
+            </gazebo>
+        </visual>
+        <xacro:box_inertial
+            mass="${scanner_mass}" length="${scanner_box_length}"
+            width="${scanner_box_width}" height="${scanner_box_height}" />
     </link>
     <!-- Materials -->
@@ -143,3 +217,12 @@
         <color rgba="0.5 0.5 0.5 1.0"/>
     </material>
+<gazebo reference="scanner_link_joint">
+    <preserveFixedJoint>true</preserveFixedJoint>
+</gazebo>
+<gazebo reference="camera_link_joint">
+    <preserveFixedJoint>true</preserveFixedJoint>
+</gazebo>
+<gazebo reference="imu_link_joint">
+    <preserveFixedJoint>true</preserveFixedJoint>
+</gazebo>
 </robot>

Commit message: convert urdf wheels to joints

File: config/urdf/r2b2.xacro (robot description, xacro)
@@ -6,9 +6,11 @@
     <xacro:property name="wheel_x_from_ctr" value="0.095" />
     <xacro:property name="wheel_y_from_ctr" value="0.0875" />
+    <xacro:property name="wheel_mass" value="0.040" />
+    <xacro:property name="wheel_max_velocity" value="${pi * 2 * (220 / 60)}" />  <!-- 220 RPM -->
     <xacro:property name="base_x_len" value="0.250" />
     <xacro:property name="base_y_width" value="0.200" />
     <xacro:property name="base_plate_ht" value="0.006" />
     <xacro:property name="base_standoff_ht" value="0.060" />
-    <xacro:property name="base_link_mass" value="2.285" />
+    <xacro:property name="base_link_mass" value="2.125" />
     <xacro:property name="motor_mount_ht" value="0.0145" />
     <xacro:property name="sensor_arch_ht" value="0.062" />
@@ -30,4 +32,5 @@
     <xacro:property name="base_box_top_ht" value="${base_box_ht_from_floor + base_box_ht}"/>
     <!-- Macros -->
+    <!-- https://en.wikipedia.org/wiki/List_of_moments_of_inertia#List_of_3D_inertia_tensors -->
     <xacro:macro name="box_inertial" params="mass length width height">
         <inertial>
@@ -43,4 +46,17 @@
         </inertial>
     </xacro:macro>
+    <xacro:macro name="cylinder_inertial" params="mass radius height">
+        <inertial>
+            <mass value="${mass}" />
+            <inertia
+                ixx="${1/12 * mass * (3 * pow(radius, 2) + pow(height, 2))}"
+                ixy="0"
+                ixz="0"
+                iyy="${1/12 * mass * (3 * pow(radius, 2) + pow(height, 2))}"
+                iyz="0"
+                izz="${1/12 * mass * pow(radius, 2)}"
+            />
+        </inertial>
+    </xacro:macro>
     <!-- Joints -->
     <joint name="camera_link_joint" type="fixed">
@@ -55,8 +71,36 @@
         <child link="imu_link"/>
     </joint>
-    <joint name="scanner_link_join" type="fixed">
+    <joint name="scanner_link_joint" type="fixed">
         <origin xyz="0.080 0 0.228" rpy="0.0 0.0 3.14159"/>
         <parent link="base_link"/>
         <child link="scanner_link"/>
+    </joint>
+    <joint name="front_left_wheel_joint" type="revolute">
+        <axis xyz="1 0 0"/>
+        <limit effort="1000.0" velocity="${wheel_max_velocity}"/>
+        <origin xyz="${wheel_x_from_ctr} ${wheel_y_from_ctr} ${wheel_dia/2}" rpy="${pi/2} 0.0 0.0"/>
+        <parent link="base_link"/>
+        <child link="front_left_wheel_link"/>
+    </joint>
+    <joint name="front_right_wheel_joint" type="revolute">
+        <axis xyz="1 0 0"/>
+        <limit effort="1000.0" velocity="${wheel_max_velocity}"/>
+        <origin xyz="${wheel_x_from_ctr} -${wheel_y_from_ctr} ${wheel_dia/2}" rpy="${pi/2} 0.0 0.0"/>
+        <parent link="base_link"/>
+        <child link="front_right_wheel_link"/>
+    </joint>
+    <joint name="rear_left_wheel_joint" type="revolute">
+        <axis xyz="1 0 0"/>
+        <limit effort="1000.0" velocity="${wheel_max_velocity}"/>
+        <origin xyz="-${wheel_x_from_ctr} ${wheel_y_from_ctr} ${wheel_dia/2}" rpy="${pi/2} 0.0 0.0"/>
+        <parent link="base_link"/>
+        <child link="rear_left_wheel_link"/>
+    </joint>
+    <joint name="rear_right_wheel_joint" type="revolute">
+        <axis xyz="1 0 0"/>
+        <limit effort="1000.0" velocity="${wheel_max_velocity}"/>
+        <origin xyz="-${wheel_x_from_ctr} -${wheel_y_from_ctr} ${wheel_dia/2}" rpy="${pi/2} 0.0 0.0"/>
+        <parent link="base_link"/>
+        <child link="rear_right_wheel_link"/>
     </joint>
     <!-- Links -->
@@ -95,45 +139,4 @@
             </gazebo>
         </visual>
-        <!-- Wheels -->
-        <visual name="front_left_wheel">
-            <geometry>
-                <cylinder radius="${wheel_dia/2}" length="${wheel_width}"/>
-            </geometry>
-            <origin xyz="${wheel_x_from_ctr} ${wheel_y_from_ctr} ${wheel_dia/2}" rpy="${pi/2} 0.0 0.0"/>
-            <material name="Black" />
-            <gazebo reference="front_left_wheel">
-                <material>Gazebo/Black</material>
-            </gazebo>
-        </visual>
-        <visual name="front_right_wheel">
-            <geometry>
-                <cylinder radius="${wheel_dia/2}" length="${wheel_width}"/>
-            </geometry>
-            <origin xyz="${wheel_x_from_ctr} -${wheel_y_from_ctr} ${wheel_dia/2}" rpy="${pi/2} 0.0 0.0"/>
-            <material name="Black" />
-            <gazebo reference="front_right_wheel">
-                <material>Gazebo/Black</material>
-            </gazebo>
-        </visual>
-        <visual name="rear_left_wheel">
-            <geometry>
-                <cylinder radius="${wheel_dia/2}" length="${wheel_width}"/>
-            </geometry>
-            <origin xyz="-${wheel_x_from_ctr} ${wheel_y_from_ctr} ${wheel_dia/2}" rpy="${pi/2} 0.0 0.0"/>
-            <material name="Black" />
-            <gazebo reference="rear_left_wheel">
-                <material>Gazebo/Black</material>
-            </gazebo>
-        </visual>
-        <visual name="rear_right_wheel">
-            <geometry>
-                <cylinder radius="${wheel_dia/2}" length="${wheel_width}"/>
-            </geometry>
-            <origin xyz="-${wheel_x_from_ctr} -${wheel_y_from_ctr} ${wheel_dia/2}" rpy="${pi/2} 0.0 0.0"/>
-            <material name="Black" />
-            <gazebo reference="rear_right_wheel">
-                <material>Gazebo/Black</material>
-            </gazebo>
-        </visual>
         <collision>
             <geometry>
@@ -145,14 +148,83 @@
             width="${base_y_width}" height="${base_box_ht}" />
     </link>
+    <!-- Wheels -->
+    <link name="front_left_wheel_link">
+        <visual name="front_left_wheel">
+            <geometry>
+                <cylinder radius="${wheel_dia/2}" length="${wheel_width}"/>
+            </geometry>
+            <material name="Black" />
+            <gazebo reference="front_left_wheel">
+                <material>Gazebo/Black</material>
+            </gazebo>
+        </visual>
+        <collision>
+            <geometry>
+                <cylinder radius="${wheel_dia/2}" length="${wheel_width}"/>
+            </geometry>
+        </collision>
+        <xacro:cylinder_inertial mass="${wheel_mass}" radius="${wheel_dia/2}" height="${wheel_width}"/>
+    </link>
+    <link name="front_right_wheel_link">
+        <visual name="front_right_wheel">
+            <geometry>
+                <cylinder radius="${wheel_dia/2}" length="${wheel_width}"/>
+            </geometry>
+            <material name="Black" />
+            <gazebo reference="front_right_wheel">
+                <material>Gazebo/Black</material>
+            </gazebo>
+        </visual>
+        <collision>
+            <geometry>
+                <cylinder radius="${wheel_dia/2}" length="${wheel_width}"/>
+            </geometry>
+        </collision>
+        <xacro:cylinder_inertial mass="${wheel_mass}" radius="${wheel_dia/2}" height="${wheel_width}"/>
+    </link>
+    <link name="rear_left_wheel_link">
+        <visual name="rear_left_wheel">
+            <geometry>
+                <cylinder radius="${wheel_dia/2}" length="${wheel_width}"/>
+            </geometry>
+            <material name="Black" />
+            <gazebo reference="rear_left_wheel">
+                <material>Gazebo/Black</material>
+            </gazebo>
+        </visual>
+        <collision>
+            <geometry>
+                <cylinder radius="${wheel_dia/2}" length="${wheel_width}"/>
+            </geometry>
+        </collision>
+        <xacro:cylinder_inertial mass="${wheel_mass}" radius="${wheel_dia/2}" height="${wheel_width}"/>
+    </link>
+    <link name="rear_right_wheel_link">
+        <visual name="rear_right_wheel">
+            <geometry>
+                <cylinder radius="${wheel_dia/2}" length="${wheel_width}"/>
+            </geometry>
+            <material name="Black" />
+            <gazebo reference="rear_right_wheel">
+                <material>Gazebo/Black</material>
+            </gazebo>
+        </visual>
+        <collision>
+            <geometry>
+                <cylinder radius="${wheel_dia/2}" length="${wheel_width}"/>
+            </geometry>
+        </collision>
+        <xacro:cylinder_inertial mass="${wheel_mass}" radius="${wheel_dia/2}" height="${wheel_width}"/>
+    </link>
     <link name="camera_link">
         <visual>
-        <geometry>
-            <box size="${camera_length}, ${camera_width} ${camera_height}"/>
-        </geometry>
-        <material name="Sky Blue" />
-        <gazebo reference="camera_link">
-            <material>Gazebo/Blue</material>
-        </gazebo>
-    </visual>
+            <geometry>
+                <box size="${camera_length}, ${camera_width} ${camera_height}"/>
+            </geometry>
+            <material name="Sky Blue" />
+            <gazebo reference="camera_link">
+                <material>Gazebo/Blue</material>
+            </gazebo>
+        </visual>
         <xacro:box_inertial
             mass="${camera_mass}" length="${camera_length}"
