Commit message: update xacro to work with gazebo

File: config/urdf/r2b2.xacro (robot description, xacro)
@@ -15,4 +15,8 @@
     <xacro:property name="motor_mount_ht" value="0.0145" />
     <xacro:property name="sensor_arch_ht" value="0.062" />
+    <!-- NUC8i5BEK 4.60" x 4.40" x 1.41" (117 mm x 112 mm x 36 mm) -->
+    <xacro:property name="nuc_length" value="0.117" />
+    <xacro:property name="nuc_width" value="0.112" />
+    <xacro:property name="nuc_height" value="0.036" />
     <xacro:property name="camera_length" value="0.025" />
     <xacro:property name="camera_width" value="0.090" />
@@ -31,4 +35,5 @@
     <xacro:property name="base_box_ht_from_floor" value="${wheel_dia/2 + motor_mount_ht}"/>
     <xacro:property name="base_box_top_ht" value="${base_box_ht_from_floor + base_box_ht}"/>
+    <xacro:property name="base_cg_height" value="${base_box_ht_from_floor + (base_box_ht + nuc_height)/2}" />
     <!-- Macros -->
     <!-- https://en.wikipedia.org/wiki/List_of_moments_of_inertia#List_of_3D_inertia_tensors -->
@@ -59,50 +64,6 @@
         </inertial>
     </xacro:macro>
-    <!-- Joints -->
-    <joint name="camera_link_joint" type="fixed">
-        <origin xyz="0.143 0.0 0.185" rpy="0.0 0.0 0.0"/>
-        <parent link="base_link"/>
-        <child link="camera_link"/>
-    </joint>
-    <joint name="imu_link_joint" type="fixed">
-        <origin xyz="0.040 -0.040 ${base_box_top_ht + sensor_arch_ht + 0.008}"
-                rpy="0.0 0.0 0.0"/>
-        <parent link="base_link"/>
-        <child link="imu_link"/>
-    </joint>
-    <joint name="scanner_link_joint" type="fixed">
-        <origin xyz="0.080 0 0.228" rpy="0.0 0.0 3.14159"/>
-        <parent link="base_link"/>
-        <child link="scanner_link"/>
-    </joint>
-    <joint name="front_left_wheel_joint" type="revolute">
-        <axis xyz="1 0 0"/>
-        <limit effort="1000.0" velocity="${wheel_max_velocity}"/>
-        <origin xyz="${wheel_x_from_ctr} ${wheel_y_from_ctr} ${wheel_dia/2}" rpy="${pi/2} 0.0 0.0"/>
-        <parent link="base_link"/>
-        <child link="front_left_wheel_link"/>
-    </joint>
-    <joint name="front_right_wheel_joint" type="revolute">
-        <axis xyz="1 0 0"/>
-        <limit effort="1000.0" velocity="${wheel_max_velocity}"/>
-        <origin xyz="${wheel_x_from_ctr} -${wheel_y_from_ctr} ${wheel_dia/2}" rpy="${pi/2} 0.0 0.0"/>
-        <parent link="base_link"/>
-        <child link="front_right_wheel_link"/>
-    </joint>
-    <joint name="rear_left_wheel_joint" type="revolute">
-        <axis xyz="1 0 0"/>
-        <limit effort="1000.0" velocity="${wheel_max_velocity}"/>
-        <origin xyz="-${wheel_x_from_ctr} ${wheel_y_from_ctr} ${wheel_dia/2}" rpy="${pi/2} 0.0 0.0"/>
-        <parent link="base_link"/>
-        <child link="rear_left_wheel_link"/>
-    </joint>
-    <joint name="rear_right_wheel_joint" type="revolute">
-        <axis xyz="1 0 0"/>
-        <limit effort="1000.0" velocity="${wheel_max_velocity}"/>
-        <origin xyz="-${wheel_x_from_ctr} -${wheel_y_from_ctr} ${wheel_dia/2}" rpy="${pi/2} 0.0 0.0"/>
-        <parent link="base_link"/>
-        <child link="rear_right_wheel_link"/>
-    </joint>
     <!-- Links -->
+    <link name="base_footprint"/>
     <link name="base_link">
         <visual name="frame_box">
@@ -111,5 +72,5 @@
                 <box size="${base_x_len} ${base_y_width} ${base_box_ht}" />
             </geometry>
-            <origin xyz="0.0 0.0 ${base_box_ht_from_floor + base_box_ht/2}"/>
+            <origin xyz="0.0 0.0 ${base_box_ht_from_floor + base_box_ht/2 - base_cg_height}"/>
             <material name="White" />
             <gazebo reference="frame_box">
@@ -120,8 +81,7 @@
             <!-- Top of NUC is 156mm from origin -->
             <geometry>
-                <!-- NUC8i5BEK 4.60" x 4.40" x 1.41" (117 mm x 112 mm x 36 mm) -->
-                <box size="0.117 0.112 0.036"/>
-            </geometry>
-            <origin xyz="-0.0335 0.0 ${base_box_top_ht + 0.036/2}"/>
+                <box size="${nuc_length} ${nuc_width} ${nuc_height}"/>
+            </geometry>
+            <origin xyz="-0.0335 0.0 ${base_box_top_ht + 0.036/2 - base_cg_height}"/>
             <material name="White" />
             <gazebo reference="nuc">
@@ -133,5 +93,5 @@
                 <box size="0.070 0.094 0.030"/>
             </geometry>
-            <origin xyz="0.077 0.0 ${base_box_top_ht + 0.030/2}"/>
+            <origin xyz="0.077 0.0 ${base_box_top_ht + 0.030/2 - base_cg_height}"/>
             <material name="White" />
             <gazebo reference="raspberry_pi4">
@@ -141,5 +101,5 @@
         <collision>
             <geometry>
-                <box size="${base_x_len} ${base_y_width} ${base_box_ht}"/>
+                <box size="${base_x_len} ${base_y_width} ${base_box_top_ht + nuc_height}"/>
             </geometry>
         </collision>
@@ -273,4 +233,50 @@
             width="${scanner_box_width}" height="${scanner_box_height}" />
     </link>
+    <!-- Joints -->
+    <joint name="base_link_joint" type="fixed">
+        <origin xyz="0 0 ${base_cg_height}" rpy="0 0 0" />
+        <parent link="base_footprint" />
+        <child link="base_link" />
+    </joint>
+    <joint name="camera_link_joint" type="fixed">
+        <origin xyz="0.143 0.0 ${0.185 - base_cg_height}" rpy="0.0 0.0 0.0"/>
+        <parent link="base_link"/>
+        <child link="camera_link"/>
+    </joint>
+    <joint name="imu_link_joint" type="fixed">
+        <origin xyz="0.040 -0.040 ${base_box_top_ht + sensor_arch_ht + 0.008 - base_cg_height}"
+                rpy="0.0 0.0 0.0"/>
+        <parent link="base_link"/>
+        <child link="imu_link"/>
+    </joint>
+    <joint name="scanner_link_joint" type="fixed">
+        <origin xyz="0.080 0 ${0.228 - base_cg_height}" rpy="0.0 0.0 3.14159"/>
+        <parent link="base_link"/>
+        <child link="scanner_link"/>
+    </joint>
+    <joint name="front_left_wheel_joint" type="continuous">
+        <axis xyz="0 0 1"/>
+        <origin xyz="${wheel_x_from_ctr} ${wheel_y_from_ctr} -${wheel_dia/2+0.1}" rpy="-${pi/2} 0.0 0.0"/>
+        <parent link="base_link"/>
+        <child link="front_left_wheel_link"/>
+    </joint>
+    <joint name="front_right_wheel_joint" type="continuous">
+        <axis xyz="0 0 1"/>
+        <origin xyz="${wheel_x_from_ctr} -${wheel_y_from_ctr} -${wheel_dia/2+0.1}" rpy="-${pi/2} 0.0 0.0"/>
+        <parent link="base_link"/>
+        <child link="front_right_wheel_link"/>
+    </joint>
+    <joint name="rear_left_wheel_joint" type="continuous">
+        <axis xyz="0 0 1"/>
+        <origin xyz="-${wheel_x_from_ctr} ${wheel_y_from_ctr} -${wheel_dia/2+0.1}" rpy="-${pi/2} 0.0 0.0"/>
+        <parent link="base_link"/>
+        <child link="rear_left_wheel_link"/>
+    </joint>
+    <joint name="rear_right_wheel_joint" type="continuous">
+        <axis xyz="0 0 1"/>
+        <origin xyz="-${wheel_x_from_ctr} -${wheel_y_from_ctr} -${wheel_dia/2+0.1}" rpy="-${pi/2} 0.0 0.0"/>
+        <parent link="base_link"/>
+        <child link="rear_right_wheel_link"/>
+    </joint>
     <!-- Materials -->
     <material name="Black">

Commit message: update robot and walls .xacro files

File: config/urdf/r2b2.xacro (robot description, xacro)
@@ -23,11 +23,15 @@
     <xacro:property name="camera_height" value="0.025" />
     <xacro:property name="camera_mass" value="0.069" />
-    <xacro:property name="scanner_box_length" value="0.0968" />
-    <xacro:property name="scanner_box_width" value="0.0703" />
-    <xacro:property name="scanner_box_height" value="0.055" />
+    <xacro:property name="scanner_length" value="0.0968" />
+    <xacro:property name="scanner_width" value="0.0703" />
+    <xacro:property name="scanner_height" value="0.057" />
+    <xacro:property name="scanner_sensor_height" value="0.048" />
+    <xacro:property name="scanner_cylinder_height" value="0.0245" />
+    <xacro:property name="scanner_cylinder_dia" value="0.070" />
     <xacro:property name="scanner_mass" value="0.170" />
     <xacro:property name="imu_length" value="0.02032" />
     <xacro:property name="imu_width" value="0.0127" />
     <xacro:property name="imu_height" value="0.003" />
+    <xacro:property name="imu_standoff_height" value="0.008" />
     <xacro:property name="imu_mass" value="0.0007" />
     <!-- Derived Measurements -->
@@ -35,5 +39,5 @@
     <xacro:property name="base_box_ht_from_floor" value="${wheel_dia/2 + motor_mount_ht}"/>
     <xacro:property name="base_box_top_ht" value="${base_box_ht_from_floor + base_box_ht}"/>
-    <xacro:property name="base_cg_height" value="${base_box_ht_from_floor + (base_box_ht + nuc_height)/2}" />
+    <xacro:property name="base_cg_height" value="${base_box_ht_from_floor + (base_box_ht/2)}" />
     <!-- Macros -->
     <!-- https://en.wikipedia.org/wiki/List_of_moments_of_inertia#List_of_3D_inertia_tensors -->
@@ -101,10 +105,109 @@
         <collision>
             <geometry>
-                <box size="${base_x_len} ${base_y_width} ${base_box_top_ht + nuc_height}"/>
+                <!-- Scanner and camera collisions ar part of their links -->
+                <!-- The base_link's collision box should be at the bottom of the motor mounts -->
+                <box size="${base_x_len} ${base_y_width - (wheel_width * 2)} ${base_box_top_ht + sensor_arch_ht - wheel_dia/2}" />
+                <!-- Translate the collision box's orgin up from the link's orgin by 1/2 of the difference in their sizes -->
+                <!-- so that they are aligned at the top, and the gap is at the bottom. -->
+                <!-- The difference in size is the wheel radius, so translate up 1/2 of the radius  -->
+                <origin xyz="0 0 ${wheel_dia/4}" rpy="0 0 0"/>
             </geometry>
         </collision>
         <xacro:box_inertial
             mass="${base_link_mass}" length="${base_x_len}"
-            width="${base_y_width}" height="${base_box_ht}" />
+            width="${base_y_width}" height="${base_box_top_ht + sensor_arch_ht}" />
+    </link>
+    <link name="camera_link">
+        <visual>
+            <geometry>
+                <box size="${camera_length}, ${camera_width} ${camera_height}"/>
+            </geometry>
+            <material name="Sky Blue" />
+            <gazebo reference="camera_link">
+                <material>Gazebo/Blue</material>
+            </gazebo>
+        </visual>
+        <collision>
+            <geometry>
+                <box size="${camera_length}, ${camera_width} ${camera_height}"/>
+            </geometry>
+        </collision>
+        <xacro:box_inertial
+            mass="${camera_mass}" length="${camera_length}"
+            width="${camera_width}" height="${camera_height}" />
+    </link>
+    <link name="imu_link">
+        <visual>
+            <geometry>
+                <box size="${imu_length} ${imu_width} ${imu_height}" />
+            </geometry>
+            <material name="PCB Green" />
+            <gazebo reference="imu_link">
+                <material>Gazebo/Green</material>
+            </gazebo>
+        </visual>
+        <collision>
+            <geometry>
+                <box size="${imu_length} ${imu_width} ${imu_height}" />
+            </geometry>
+        </collision>
+        <xacro:box_inertial
+            mass="${imu_mass}" length="${imu_length}"
+            width="${imu_width}" height="${imu_height}" />
+    </link>
+    <link name="scanner_link">
+        <!-- Note: Scanner link's origin needs to be where the receive sensor is located, near the top -->
+        <visual name="scanner_cylinder_visual">
+            <geometry>
+                <cylinder radius="${scanner_cylinder_dia/2}" length="${scanner_cylinder_height}"/>
+            </geometry>
+            <!--
+                Rotating cylinder is 24.5mm tall
+                Receive sensor origin is 15.5mm above bottom of cylinder:
+                    i.e. scanner_sensor_height - (scanner_height - scanner_cylinder_height)
+                So the cylinder visual should be dropped by the difference
+                    y = (24.5/2) - 15.5 = -3.25mm
+            -->
+            <origin xyz="0 0 ${scanner_cylinder_height/2 - (scanner_sensor_height - (scanner_height - scanner_cylinder_height))}"/>
+            <material name="Black" />
+            <gazebo reference="scanner_cylinder_visual">
+                <material>Gazebo/Orange</material>
+            </gazebo>
+        </visual>
+        <visual name="scanner_box_visual">
+            <geometry>
+                <box size="${scanner_length} ${scanner_width} ${scanner_height - scanner_cylinder_height}"/>
+            </geometry>
+            <!-- <origin xyz="0.015 0.0 -0.033"/> -->
+            <!--
+                Calculate the visual origin of the base box which sits under the cylinder.
+                X:
+                Align the front edge. So just translate by the difference on one side
+                Which = (Xscanner - Xcylinder)/2 since the difference is on each side
+                Y: No change since the scanner is in the center of base
+                Z:
+                This is the simplified expression of the longer calculation
+                -(Hbox/2 + (Hcylinder - (Hscanner - Hsensor)))
+                Where Hbox = Hscanner - Hcylinder
+            -->
+            <origin xyz="${(scanner_length - scanner_cylinder_dia)/2} 0.0 ${ -(scanner_cylinder_height - scanner_height + (2 * scanner_sensor_height)) / 2 }" />
+            <material name="Black" />
+            <gazebo reference="scanner_box_visual">
+                <material>Gazebo/Black</material>
+            </gazebo>
+        </visual>
+        <collision>
+            <!--
+            The collision box needs to be dropped from the sensor origin,
+            since the sensor origin is near the top of the scanner box.
+            -->
+            <origin xyz="0.0 0.0 ${scanner_height/2 - (scanner_height - scanner_sensor_height)}"/>
+            <geometry>
+                <box size="${scanner_length} ${scanner_width} ${scanner_height}"/>
+            </geometry>
+        </collision>
+        <xacro:box_inertial
+            mass="${scanner_mass}" length="${scanner_length}"
+            width="${scanner_width}" height="${scanner_height}" />
     </link>
     <!-- Wheels -->
@@ -176,60 +279,4 @@
         </collision>
         <xacro:cylinder_inertial mass="${wheel_mass}" radius="${wheel_dia/2}" height="${wheel_width}"/>
-    </link>
-    <link name="camera_link">
-        <visual>
-            <geometry>
-                <box size="${camera_length}, ${camera_width} ${camera_height}"/>
-            </geometry>
-            <material name="Sky Blue" />
-            <gazebo reference="camera_link">
-                <material>Gazebo/Blue</material>
-            </gazebo>
-        </visual>
-        <xacro:box_inertial
-            mass="${camera_mass}" length="${camera_length}"
-            width="${camera_width}" height="${camera_height}" />
-    </link>
-    <link name="imu_link">
-        <visual>
-            <geometry>
-                <box size="${imu_length} ${imu_width} ${imu_height}" />
-            </geometry>
-            <material name="PCB Green" />
-            <gazebo reference="imu_link">
-                <material>Gazebo/Green</material>
-            </gazebo>
-        </visual>
-        <xacro:box_inertial
-            mass="${imu_mass}" length="${imu_length}"
-            width="${imu_width}" height="${imu_height}" />
-    </link>
-    <link name="scanner_link">
-        <visual>
-            <geometry>
-                <!--
-                    Rotating cylinder is 24mm tall
-                    Receive sensor is 16.5mm above bottom surface
-                    So the visual should be dropped by the difference
-                        y = (24/2) - 16.5 = -4.5mm
-                -->
-                <cylinder radius="0.035" length="0.024"/>
-            </geometry>
-            <origin xyz="0 0 -0.0045"/>
-            <material name="Black" />
-        </visual>
-        <visual>
-            <geometry>
-                <box size="0.100 0.070 0.033"/>
-            </geometry>
-            <origin xyz="0.015 0.0 -0.033"/>
-            <material name="Black" />
-            <gazebo reference="scanner_link">
-                <material>Gazebo/Black</material>
-            </gazebo>
-        </visual>
-        <xacro:box_inertial
-            mass="${scanner_mass}" length="${scanner_box_length}"
-            width="${scanner_box_width}" height="${scanner_box_height}" />
     </link>
     <!-- Joints -->
@@ -245,5 +292,5 @@
     </joint>
     <joint name="imu_link_joint" type="fixed">
-        <origin xyz="0.040 -0.040 ${base_box_top_ht + sensor_arch_ht + 0.008 - base_cg_height}"
+        <origin xyz="0.040 -0.040 ${base_box_top_ht + sensor_arch_ht + imu_standoff_height - base_cg_height}"
                 rpy="0.0 0.0 0.0"/>
         <parent link="base_link"/>
@@ -257,5 +304,5 @@
     <joint name="front_left_wheel_joint" type="continuous">
         <axis xyz="0 0 1"/>
-        <origin xyz="${wheel_x_from_ctr} ${wheel_y_from_ctr} -${wheel_dia/2+0.1}" rpy="-${pi/2} 0.0 0.0"/>
+        <origin xyz="${wheel_x_from_ctr} ${wheel_y_from_ctr} ${wheel_dia/2 - base_cg_height}" rpy="-${pi/2} 0.0 0.0"/>
         <parent link="base_link"/>
         <child link="front_left_wheel_link"/>
@@ -263,5 +310,5 @@
     <joint name="front_right_wheel_joint" type="continuous">
         <axis xyz="0 0 1"/>
-        <origin xyz="${wheel_x_from_ctr} -${wheel_y_from_ctr} -${wheel_dia/2+0.1}" rpy="-${pi/2} 0.0 0.0"/>
+        <origin xyz="${wheel_x_from_ctr} -${wheel_y_from_ctr} ${wheel_dia/2 - base_cg_height}" rpy="-${pi/2} 0.0 0.0"/>
         <parent link="base_link"/>
         <child link="front_right_wheel_link"/>
@@ -269,5 +316,5 @@
     <joint name="rear_left_wheel_joint" type="continuous">
         <axis xyz="0 0 1"/>
-        <origin xyz="-${wheel_x_from_ctr} ${wheel_y_from_ctr} -${wheel_dia/2+0.1}" rpy="-${pi/2} 0.0 0.0"/>
+        <origin xyz="-${wheel_x_from_ctr} ${wheel_y_from_ctr} ${wheel_dia/2 - base_cg_height}" rpy="-${pi/2} 0.0 0.0"/>
         <parent link="base_link"/>
         <child link="rear_left_wheel_link"/>
@@ -275,5 +322,5 @@
     <joint name="rear_right_wheel_joint" type="continuous">
         <axis xyz="0 0 1"/>
-        <origin xyz="-${wheel_x_from_ctr} -${wheel_y_from_ctr} -${wheel_dia/2+0.1}" rpy="-${pi/2} 0.0 0.0"/>
+        <origin xyz="-${wheel_x_from_ctr} -${wheel_y_from_ctr} ${wheel_dia/2 - base_cg_height}" rpy="-${pi/2} 0.0 0.0"/>
         <parent link="base_link"/>
         <child link="rear_right_wheel_link"/>

Commit message: add gazebo lidar and depth camera

File: config/urdf/r2b2.xacro (robot description, xacro)
@@ -136,5 +136,5 @@
             mass="${camera_mass}" length="${camera_length}"
             width="${camera_width}" height="${camera_height}" />
-    </link>
+     </link>
     <link name="imu_link">
         <visual>
@@ -342,12 +342,60 @@
         <color rgba="0.5 0.5 0.5 1.0"/>
     </material>
-<gazebo reference="scanner_link_joint">
-    <preserveFixedJoint>true</preserveFixedJoint>
-</gazebo>
-<gazebo reference="camera_link_joint">
-    <preserveFixedJoint>true</preserveFixedJoint>
-</gazebo>
-<gazebo reference="imu_link_joint">
-    <preserveFixedJoint>true</preserveFixedJoint>
-</gazebo>
+    <gazebo reference="scanner_link_joint">
+        <preserveFixedJoint>true</preserveFixedJoint>
+    </gazebo>
+    <gazebo reference="camera_link_joint">
+        <preserveFixedJoint>true</preserveFixedJoint>
+    </gazebo>
+    <gazebo reference="imu_link_joint">
+        <preserveFixedJoint>true</preserveFixedJoint>
+    </gazebo>
+    <gazebo reference="scanner_link">
+        <sensor name='gpu_lidar' type='gpu_lidar'>
+            <pose relative_to="scanner_link">0 0 0 0 0 0</pose>
+            <topic>lidar</topic>
+            <update_rate>10</update_rate>
+            <lidar>
+                <scan>
+                <horizontal>
+                    <samples>640</samples>
+                    <resolution>1</resolution>
+                    <min_angle>-1.396263</min_angle>
+                    <max_angle>1.396263</max_angle>
+                </horizontal>
+                <vertical>
+                    <samples>16</samples>
+                    <resolution>1</resolution>
+                    <min_angle>-0.261799</min_angle>
+                    <max_angle>0.261799</max_angle>
+                </vertical>
+                </scan>
+                <range>
+                <min>0.08</min>
+                <max>10.0</max>
+                <resolution>0.01</resolution>
+                </range>
+            </lidar>
+            <always_on>true</always_on>
+            <visualize>true</visualize>
+        </sensor>
+    </gazebo>
+    <gazebo reference="camera_link">
+        <sensor name="realsense_d435" type="depth_camera">
+            <update_rate>10</update_rate>
+            <topic>depth_camera</topic>
+            <camera>
+              <horizontal_fov>1.05</horizontal_fov>
+              <image>
+                <width>256</width>
+                <height>256</height>
+                <format>R_FLOAT32</format>
+              </image>
+              <clip>
+                <near>0.1</near>
+                <far>10.0</far>
+              </clip>
+            </camera>
+        </sensor>
+    </gazebo>
 </robot>
