Commit message: add r2b2.launch.py

File: config/urdf/r2b2.xacro (robot description, xacro)
@@ -121,5 +121,5 @@
         <visual>
             <geometry>
-                <box size="${camera_length}, ${camera_width} ${camera_height}"/>
+                <box size="${camera_length} ${camera_width} ${camera_height}"/>
             </geometry>
             <material name="Sky Blue" />
@@ -130,5 +130,5 @@
         <collision>
             <geometry>
-                <box size="${camera_length}, ${camera_width} ${camera_height}"/>
+                <box size="${camera_length} ${camera_width} ${camera_height}"/>
             </geometry>
         </collision>
@@ -157,5 +157,5 @@
     </link>
     <link name="scanner_link">
-        <!-- Note: Scanner link's origin needs to be where the receive sensor is located, near the top -->
+        <!-- Note Scanner link's origin needs to be where the receive sensor is located, near the top -->
         <visual name="scanner_cylinder_visual">
             <geometry>
@@ -164,5 +164,5 @@
             <!--
                 Rotating cylinder is 24.5mm tall
-                Receive sensor origin is 15.5mm above bottom of cylinder:
+                Receive sensor origin is 15.5mm above bottom of cylinder
                     i.e. scanner_sensor_height - (scanner_height - scanner_cylinder_height)
                 So the cylinder visual should be dropped by the difference
@@ -182,9 +182,9 @@
             <!--
                 Calculate the visual origin of the base box which sits under the cylinder.
-                X:
+                X-
                 Align the front edge. So just translate by the difference on one side
                 Which = (Xscanner - Xcylinder)/2 since the difference is on each side
-                Y: No change since the scanner is in the center of base
-                Z:
+                Y- No change since the scanner is in the center of base
+                Z-
                 This is the simplified expression of the longer calculation
                 -(Hbox/2 + (Hcylinder - (Hscanner - Hsensor)))
@@ -352,7 +352,7 @@
     </gazebo>
     <gazebo reference="scanner_link">
-        <sensor name='gpu_lidar' type='gpu_lidar'>
+        <sensor name='rplidar_a1' type='gpu_lidar'>
             <pose relative_to="scanner_link">0 0 0 0 0 0</pose>
-            <topic>lidar</topic>
+            <topic>scan</topic>
             <update_rate>10</update_rate>
             <lidar>

Commit message: update launch and config files for sim nav

File: config/urdf/r2b2.xacro (robot description, xacro)
@@ -191,5 +191,5 @@
                 Where Hbox = Hscanner - Hcylinder
             -->
-            <origin xyz="${(scanner_length - scanner_cylinder_dia)/2} 0.0 ${ -(scanner_cylinder_height - scanner_height + (2 * scanner_sensor_height)) / 2 }" />
+            <origin xyz="${-(scanner_length - scanner_cylinder_dia)/2} 0.0 ${ -(scanner_cylinder_height - scanner_height + (2 * scanner_sensor_height)) / 2 }" />
             <material name="Black" />
             <gazebo reference="scanner_box_visual">
@@ -298,5 +298,5 @@
     </joint>
     <joint name="scanner_link_joint" type="fixed">
-        <origin xyz="0.080 0 ${0.228 - base_cg_height}" rpy="0.0 0.0 3.14159"/>
+        <origin xyz="0.080 0 ${0.228 - base_cg_height}" rpy="0.0 0.0 0.0"/>
         <parent link="base_link"/>
         <child link="scanner_link"/>
@@ -353,4 +353,5 @@
     <gazebo reference="scanner_link">
         <sensor name='rplidar_a1' type='gpu_lidar'>
+            <!-- 10Hz @ 4000 points = 400 samples and 10 update rate -->
             <pose relative_to="scanner_link">0 0 0 0 0 0</pose>
             <topic>scan</topic>
@@ -358,22 +359,31 @@
             <lidar>
                 <scan>
-                <horizontal>
-                    <samples>640</samples>
-                    <resolution>1</resolution>
-                    <min_angle>-1.396263</min_angle>
-                    <max_angle>1.396263</max_angle>
-                </horizontal>
-                <vertical>
-                    <samples>16</samples>
-                    <resolution>1</resolution>
-                    <min_angle>-0.261799</min_angle>
-                    <max_angle>0.261799</max_angle>
-                </vertical>
-                </scan>
+                    <horizontal>
+                        <samples>400</samples>
+                        <resolution>1</resolution>
+                        <min_angle>-${pi}</min_angle>
+                        <max_angle>${pi}</max_angle>
+                    </horizontal>
+                    <vertical>
+                        <!-- <samples>16</samples>
+                        <resolution>1</resolution>
+                        <min_angle>-0.261799</min_angle>
+                        <max_angle>0.261799</max_angle> -->
+                        <samples>3</samples>
+                        <resolution>1</resolution>
+                        <min_angle>-0.261799</min_angle>
+                        <max_angle>0.261799</max_angle>
+                    </vertical>
+                    </scan>
                 <range>
-                <min>0.08</min>
-                <max>10.0</max>
-                <resolution>0.01</resolution>
+                    <min>0.15</min>
+                    <max>12.0</max>
+                    <resolution>0.01</resolution>
                 </range>
+                <noise>
+                    <type>guassian</type>
+                    <mean>0.0</mean>
+                    <stddev>0.01</stddev>
+                </noise>
             </lidar>
             <always_on>true</always_on>

Commit message: update nav and gazebo

File: config/urdf/r2b2.xacro (robot description, xacro)
@@ -287,5 +287,5 @@
     </joint>
     <joint name="camera_link_joint" type="fixed">
-        <origin xyz="0.143 0.0 ${0.185 - base_cg_height}" rpy="0.0 0.0 0.0"/>
+        <origin xyz="0.143 0.0 ${0.185 - base_cg_height}" rpy="0.0 0.3491 0.0"/>
         <parent link="base_link"/>
         <child link="camera_link"/>
@@ -393,19 +393,130 @@
     </gazebo>
     <gazebo reference="camera_link">
-        <!-- <sensor name="realsense_d435_depth" type="depth_camera">
-            <topic>depth_camera</topic>
-            <update_rate>10</update_rate>
+        <sensor name="rgbd_camera" type="rgbd_camera">
+            <topic>rgbd_camera</topic>
+            <update_rate>30</update_rate>
+            <camera>
+                <horizontal_fov>1.2133529</horizontal_fov>
+                <image>
+                    <width>640</width>
+                    <height>480</height>
+                    <format>R8G8B8</format>
+                </image>
+                <distortion>
+                    <k1>0</k1>
+                    <k2>0</k2>
+                    <k3>0</k3>
+                    <p1>0</p1>
+                    <p2>0</p2>
+                    <center>0.5 0.5</center>
+                </distortion>
+                <lens>
+                    <type>sterographic</type>
+                    <scale_to_hfov>true</scale_to_hfov>
+                    <intrinsics>
+                        <fx>461.115600585938</fx>
+                        <fy>461.144226074219</fy>
+                        <cx>319.159820556641</cx>
+                        <cy>181.155624389648</cy>
+                        <s>0</s>
+                    </intrinsics>
+                </lens>
+                <clip>
+                    <near>0.1</near>
+                    <far>50</far>
+                </clip>
+            </camera>
             <depth_camera>
-              <horizontal_fov>1.05</horizontal_fov>
-              <image>
-                <width>256</width>
-                <height>256</height>
-                <format>R_FLOAT32</format>
-              </image>
-              <clip>
-                <near>0.1</near>
-                <far>10.0</far>
+                <output>depths</output>
+                <clip>
+                    <near>0.3</near>
+                    <far>3.0</far>
+                </clip>
+            </depth_camera>
+            <always_on>1</always_on>
+            <visualize>true</visualize>
+            <enable_metrics>true</enable_metrics>
+            <ignition_frame_id>camera_link</ignition_frame_id>
+          </sensor>
+        <!-- <sensor name="realsense_D435_rgb" type="camera">
+            <topic>realsense/color/image_raw</topic>
+            <update_rate>30</update_rate>
+            <camera>
+                <horizontal_fov>1.2133529</horizontal_fov>
+                <image>
+                    <width>640</width>
+                    <height>360</height>
+                    <format>R8G8B8</format>
+                </image>
+                <distortion>
+                    <k1>0</k1>
+                    <k2>0</k2>
+                    <k3>0</k3>
+                    <p1>0</p1>
+                    <p2>0</p2>
+                    <center>0.5 0.5</center>
+                </distortion>
+                <lens>
+                    <type>sterographic</type>
+                    <scale_to_hfov>true</scale_to_hfov>
+                    <intrinsics>
+                        <fx>461.115600585938</fx>
+                        <fy>461.144226074219</fy>
+                        <cx>319.159820556641</cx>
+                        <cy>181.155624389648</cy>
+                        <s>0</s>
+                    </intrinsics>
+                </lens>
+            </camera>
+            <always_on>1</always_on>
+            <visualize>true</visualize>
+            <ignition_frame_id>camera_link</ignition_frame_id>
+        </sensor> -->
+        <!-- Intrinsic of "Color" / 640x360 / {YUYV/RGB8/BGR8/RGBA8/BGRA8/Y16}
+        Width:      	640
+        Height:     	360
+        PPX:        	319.159820556641
+        PPY:        	181.155624389648
+        Fx:         	461.115600585938
+        Fy:         	461.144226074219
+        Distortion: 	Inverse Brown Conrady
+        Coeffs:     	0  	0  	0  	0  	0
+        FOV (deg):  	69.52 x 42.64 -->
+        <!-- <sensor name="realsense_D435_depth" type="depth_camera">
+            <topic>realsense/depth/image_rect_raw</topic>
+            <update_rate>6</update_rate>
+            <camera>
+                <horizontal_fov>1.5610225</horizontal_fov>
+                <image>
+                    <width>640</width>
+                    <height>360</height>
+                    <format>R_FLOAT32</format>
+                </image>
+                <distortion>
+                    <k1>0</k1>
+                    <k2>0</k2>
+                    <k3>0</k3>
+                    <p1>0</p1>
+                    <p2>0</p2>
+                    <center>0.5 0.5</center>
+                </distortion>
+                <lens>
+                    <type>sterographic</type>
+                    <scale_to_hfov>true</scale_to_hfov>
+                    <intrinsics>
+                        <fx>323.143859863281</fx>
+                        <fy>323.143859863281</fy>
+                        <cx>317.321014404297</cx>
+                        <cy>177.92724609375</cy>
+                        <s>0</s>
+                    </intrinsics>
+                </lens>
+            </camera>
+            <depth_camera>
+                <output>depths</output>
+                <clip>
+                <near>0.3</near>
+                <far>3.0</far>
               </clip>
-              <output>depths</output>
             </depth_camera>
             <always_on>1</always_on>
@@ -413,41 +524,14 @@
             <ignition_frame_id>camera_link</ignition_frame_id>
         </sensor> -->
-        <!-- <sensor name="realsense_d435_rgb" type="camera">
-            <topic>rgb_camera</topic>
-            <update_rate>30</update_rate>
-            <camera>
-              <horizontal_fov>1.047</horizontal_fov>
-              <image>
-                <width>320</width>
-                <height>240</height>
-              </image>
-              <clip>
-                <near>0.1</near>
-                <far>100</far>
-              </clip>
-            </camera>
-            <always_on>1</always_on>
-            <visualize>true</visualize>
-            <ignition_frame_id>camera_link</ignition_frame_id>
-        </sensor>         -->
-        <sensor name="rgbd_camera" type="rgbd_camera">
-            <topic>rgbd_camera</topic>
-            <update_rate>30</update_rate>
-            <camera>
-              <horizontal_fov>1.047</horizontal_fov>
-              <image>
-                <width>320</width>
-                <height>240</height>
-              </image>
-              <clip>
-                <near>0.1</near>
-                <far>100</far>
-              </clip>
-            </camera>
-            <always_on>1</always_on>
-            <visualize>true</visualize>
-            <enable_metrics>true</enable_metrics>
-            <ignition_frame_id>camera_link</ignition_frame_id>
-          </sensor>
+        <!-- Intrinsic of "Depth" / 640x360 / {Z16}
+        Width:      	640
+        Height:     	360
+        PPX:        	317.321014404297
+        PPY:        	177.92724609375
+        Fx:         	323.143859863281
+        Fy:         	323.143859863281
+        Distortion: 	Brown Conrady
+        Coeffs:     	0  	0  	0  	0  	0
+        FOV (deg):  	89.44 x 58.24 -->
     </gazebo>
     <gazebo reference="imu_link">

Commit message: adjustments to r2b2 runtime launch config

File: config/urdf/r2b2.xacro (robot description, xacro)
@@ -191,5 +191,5 @@
                 Where Hbox = Hscanner - Hcylinder
             -->
-            <origin xyz="${-(scanner_length - scanner_cylinder_dia)/2} 0.0 ${ -(scanner_cylinder_height - scanner_height + (2 * scanner_sensor_height)) / 2 }" />
+            <origin xyz="${(scanner_length - scanner_cylinder_dia)/2} 0.0 ${ -(scanner_cylinder_height - scanner_height + (2 * scanner_sensor_height)) / 2 }" />
             <material name="Black" />
             <gazebo reference="scanner_box_visual">
@@ -287,5 +287,6 @@
     </joint>
     <joint name="camera_link_joint" type="fixed">
-        <origin xyz="0.143 0.0 ${0.185 - base_cg_height}" rpy="0.0 0.3491 0.0"/>
+        <!-- <origin xyz="0.143 0.0 ${0.185 - base_cg_height}" rpy="0.0 0.3491 0.0"/> -->
+        <origin xyz="0.143 0.0 ${0.185 - base_cg_height}" rpy="0.0 0.0 0.0"/>
         <parent link="base_link"/>
         <child link="camera_link"/>
@@ -298,5 +299,12 @@
     </joint>
     <joint name="scanner_link_joint" type="fixed">
-        <origin xyz="0.080 0 ${0.228 - base_cg_height}" rpy="0.0 0.0 0.0"/>
+        <!--
+            The RPLidar A1 has the 0-deg angle opposite of the X-axis. In other words, the motor
+            is in front be desitn. But we have the motor in the back. So we need to rotate the joint
+            by 180-deg on the actual robot.
+            However, in Gazebo the laser scan plugin has 0-deg on the x-axis. So we don't need to
+            rotate it.
+            -->
+        <origin xyz="0.080 0 ${0.228 - base_cg_height}" rpy="0.0 0.0 ${pi}"/>
         <parent link="base_link"/>
         <child link="scanner_link"/>
